File: pcb/chocopi.kicad_sch (KiCad schematic)
At the start: 39 parts, among them U1 XIAO-nRF52840-SMD

Commit message: positioned
Parts:
- added BAT+2: +, chocopi:BatteryPad, symbol Mechanical:MountingHole_Pad
- added BATGND2: -, chocopi:BatteryPad, symbol Mechanical:MountingHole_Pad
- added PSW2: SW_SPDT, chocopi:MSK12C02, symbol Switch:SW_SPDT
- added S2: EVQ-P7A01P, chocopi:SW_EVQ-P7A01P, symbol EVQ-P7A01P:EVQ-P7A01P
- added U2: XIAO-nRF52840-SMD, chocopi:xiao-ble-smd-cutout, symbol chocopi:xiao
- added r_D1, r_D10, r_D11, r_D12, r_D13, r_D14, r_D15, r_D16, r_D17, r_D2, r_D3, r_D4, r_D5, r_D6, r_D7, r_D8, r_D9: ~, chocopi:Diode_SOD123, symbol chocopi:d
- added r_sw1, r_sw10, r_sw11, r_sw12, r_sw13, r_sw14, r_sw15, r_sw16, r_sw17, r_sw2, r_sw3, r_sw4, r_sw5, r_sw6, r_sw7, r_sw8, r_sw9: ~, chocopi:Cherry_ULP_SMD, symbol chocopi:sw
- renumbered sw1 to swl1
Connections:
- net BAT+ renamed l_BAT+
- net GND renamed l_GND
- net RESET renamed l_RESET
- net VBAT renamed l_VBAT
- net col1 renamed l_col1
- net col2 renamed l_col2
- net col3 renamed l_col3
- net col4 renamed l_col4
- net col5 renamed l_col5
- net row1 renamed l_row1
- net row2 renamed l_row2
- net row3 renamed l_row3
- net row4 renamed l_row4
- new net: r_D10.1 (K), r_sw10.2
- new net: r_D8.1 (K), r_sw8.2
- new net: r_D4.1 (K), r_sw4.2
- new net: r_D9.1 (K), r_sw9.2
- new net: r_D7.1 (K), r_sw7.2
- new net: r_D17.1 (K), r_sw17.2
- new net: r_D14.1 (K), r_sw14.2
- new net: r_D6.1 (K), r_sw6.2
- new net: r_D5.1 (K), r_sw5.2
- new net: r_D2.1 (K), r_sw2.2
- new net: r_D11.1 (K), r_sw11.2
- new net: r_D12.1 (K), r_sw12.2
- new net: r_D16.1 (K), r_sw16.2
- new net: r_D3.1 (K), r_sw3.2
- new net: r_D15.1 (K), r_sw15.2
- new net: r_D13.1 (K), r_sw13.2
- new net: r_D1.1 (K), r_sw1.2
- new net r_BAT+: PSW2.2 (B), U2.19 (BAT)
- new net r_GND: BATGND2.1, S2.2_1, S2.2_2, U2.13 (GND), U2.18 (GND), U2.20 (GND)
- new net r_RESET: S2.1_1, S2.1_2, U2.17 (RESET)
- new net r_VBAT: BAT+2.1, PSW2.3 (C)
- new net r_col1: U2.5 (A8_SDA/0.04_H), r_sw1.1, r_sw11.1, r_sw16.1, r_sw6.1
- new net r_col2: U2.6 (A9_SCL/0.05_H), r_sw12.1, r_sw17.1, r_sw2.1, r_sw7.1
- new net r_col3: U2.11 (A6_MOSI/1.15), r_sw13.1, r_sw3.1, r_sw8.1
- new net r_col4: U2.10 (A5_MISO/1.14), r_sw14.1, r_sw4.1, r_sw9.1
- new net r_col5: U2.9 (A7_SCK/1.13), r_sw10.1, r_sw15.1, r_sw5.1
- new net r_row1: U2.1 (A2/0.02_H), r_D1.2 (A), r_D2.2 (A), r_D3.2 (A), r_D4.2 (A), r_D5.2 (A)
- new net r_row2: r_D10.2 (A), r_D6.2 (A), r_D7.2 (A), r_D8.2 (A), r_D9.2 (A)
- new net r_row2 : U2.2 (A4/0.03_H)
- new net r_row3: U2.3 (A10/0.28), r_D11.2 (A), r_D12.2 (A), r_D13.2 (A), r_D14.2 (A), r_D15.2 (A)
- new net r_row4: U2.4 (A11/0.29), r_D16.2 (A), r_D17.2 (A)
- no-connect marks 6 -> 12
Other:
- moved on the sheet: BAT+1, BATGND1, PSW1, S1
