File: pcb/chocopi.kicad_pcb (KiCad board)
At the start: 2 copper layers, 114.3 x 93 mm, 39 parts, among them U1 XIAO-nRF52840-SMD

Commit message: fix diode
Parts:
- moved D16 7.21 mm to (121.8, 80.6)
Routing:
- net row4: track 22.4 -> 29.8 mm
- net Net-(D16-K): track 6.86 -> 12.8 mm
Changed lines of the file:
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@@
 		(placed yes)
 		(layer "B.Cu")
-		(at 129 81)
+		(at 121.8 80.6)
 		(descr "Diode, DO-41, SOD81, Horizontal, RM 10mm,")
 		(tags "Diode, DO-41, SOD81, Horizontal, RM 10mm, 1N4007, SB140,")
@@
 	)
 	(segment
-		(start 127.3 83.5)
-		(end 127.3 81)
+		(start 128.4 84.6)
+		(end 127.3 83.5)
 		(width 0.2)
 		(layer "B.Cu")
@@
 	)
 	(segment
-		(start 128.4 84.6)
+		(start 120.1 80.6)
+		(end 123 83.5)
+		(width 0.2)
+		(layer "B.Cu")
+		(net 19)
+	)
+	(segment
+		(start 123 83.5)
 		(end 127.3 83.5)
 		(width 0.2)
@@
 	)
 	(segment
-		(start 130.7 81)
-		(end 131.088154 81.388154)
+		(start 123.5 80.6)
+		(end 130.3 80.6)
 		(width 0.2)
 		(layer "B.Cu")
@@
 		(width 0.2)
 		(layer "B.Cu")
+		(net 20)
+	)
+	(segment
+		(start 130.3 80.6)
+		(end 131.088154 81.388154)
+		(width 0.2)
+		(layer "B.Cu")

Commit message: wip
Parts:
- moved D13 22.8 mm to (75.7, 55.9)
- moved D12 4.90 mm to (75.7, 59.4)
Routing:
- net Net-(D13-K): track 0.00 -> 26.1 mm, vias 1 -> 3
- net Net-(D12-K): track 0.00 -> 6.70 mm
- net row3: track 168.7 -> 162.4 mm
- net col2: track 154.2 -> 153.2 mm
- net col1: track 156.6 -> 155.9 mm

Commit message: positioned
Parts:
- added BAT+2: +, chocopi:BatteryPad, F.Cu at (270.7, 153.3)
- added BATGND2: -, chocopi:BatteryPad, F.Cu at (270.7, 156.8)
- added PSW2: SW_SPDT, chocopi:MSK12C02, B.Cu at (184.2, 68.7)
- added S2: EVQ-P7A01P, chocopi:SW_EVQ-P7A01P, B.Cu at (185.7, 82.1)
- added U2: XIAO-nRF52840-SMD, chocopi:xiao-ble-smd-cutout, B.Cu at (187.9, 103.7)
- added r_D1: ~, chocopi:Diode_SOD123, F.Cu at (267.1, 137.5)
- added r_D10: ~, chocopi:Diode_SOD123, F.Cu at (273.3, 145.2)
- added r_D11: ~, chocopi:Diode_SOD123, F.Cu at (273.3, 147.7)
- added r_D12: ~, chocopi:Diode_SOD123, F.Cu at (273.3, 150.3)
- added r_D13: ~, chocopi:Diode_SOD123, F.Cu at (279.5, 137.5)
- added r_D14: ~, chocopi:Diode_SOD123, F.Cu at (279.5, 140.1)
- added r_D15: ~, chocopi:Diode_SOD123, F.Cu at (279.5, 142.6)
- added r_D16: ~, chocopi:Diode_SOD123, F.Cu at (279.5, 145.2)
- added r_D17: ~, chocopi:Diode_SOD123, F.Cu at (279.5, 147.7)
- added r_D2: ~, chocopi:Diode_SOD123, F.Cu at (267.1, 140.1)
- added r_D3: ~, chocopi:Diode_SOD123, F.Cu at (267.1, 142.6)
- added r_D4: ~, chocopi:Diode_SOD123, F.Cu at (267.1, 145.2)
- added r_D5: ~, chocopi:Diode_SOD123, F.Cu at (267.1, 147.7)
- added r_D6: ~, chocopi:Diode_SOD123, F.Cu at (267.1, 150.3)
- added r_D7: ~, chocopi:Diode_SOD123, F.Cu at (273.3, 137.5)
- added r_D8: ~, chocopi:Diode_SOD123, F.Cu at (273.3, 140.1)
- added r_D9: ~, chocopi:Diode_SOD123, F.Cu at (273.3, 142.6)
- added r_sw1: ~, chocopi:Cherry_ULP_SMD, F.Cu at (193.3, 56.4)
- added r_sw10: ~, chocopi:Cherry_ULP_SMD, F.Cu at (267.4, 83.0)
- added r_sw11: ~, chocopi:Cherry_ULP_SMD, F.Cu at (193.3, 91.4)
- added r_sw12: ~, chocopi:Cherry_ULP_SMD, F.Cu at (211.8, 88.7)
- added r_sw13: ~, chocopi:Cherry_ULP_SMD, F.Cu at (230.3, 82.5)
- added r_sw14: ~, chocopi:Cherry_ULP_SMD, F.Cu at (248.9, 88.5)
- added r_sw15: ~, chocopi:Cherry_ULP_SMD, F.Cu at (267.4, 100.5)
- added r_sw16: ~, chocopi:Cherry_ULP_SMD, F.Cu at (198.3, 111.6)
- added r_sw17: ~, chocopi:Cherry_ULP_SMD, F.Cu at (176.6, 115.7)
- added r_sw2: ~, chocopi:Cherry_ULP_SMD, F.Cu at (211.8, 53.7)
- added r_sw3: ~, chocopi:Cherry_ULP_SMD, F.Cu at (230.3, 47.4)
- added r_sw4: ~, chocopi:Cherry_ULP_SMD, F.Cu at (248.9, 53.4)
- added r_sw5: ~, chocopi:Cherry_ULP_SMD, F.Cu at (267.4, 65.4)
- added r_sw6: ~, chocopi:Cherry_ULP_SMD, F.Cu at (193.3, 73.9)
- added r_sw7: ~, chocopi:Cherry_ULP_SMD, F.Cu at (211.8, 71.2)
- added r_sw8: ~, chocopi:Cherry_ULP_SMD, F.Cu at (230.3, 65.0)
- added r_sw9: ~, chocopi:Cherry_ULP_SMD, F.Cu at (248.9, 70.9)
- moved U1 34.7 mm to (116.3, 103.8)
- moved D12 34.4 mm to (54.9, 86.7)
- moved D13 34.4 mm to (54.9, 83.2)
- moved D16 34.4 mm to (101.0, 107.9)
- moved sw17 34.4 mm to (127.6, 115.8)
- moved BAT+1 34.4 mm to (101.2, 80.8)
- moved BATGND1 34.4 mm to (101.2, 84.3)
- moved D1 34.4 mm to (40.2, 66.8)
- moved D10 34.4 mm to (114.2, 75.3)
- moved D11 34.4 mm to (40.2, 101.8)
- moved D14 34.4 mm to (95.7, 90.3)
- moved D15 34.4 mm to (110.9, 88.8)
- moved D17 34.4 mm to (128.2, 112.8)
- moved D2 34.4 mm to (58.7, 54.8)
- moved D3 34.4 mm to (77.2, 48.8)
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- renumbered sw1 to swl1
Connections:
- net BAT+ renamed l_BAT+
- net GND renamed l_GND
- net RESET renamed l_RESET
- net VBAT renamed l_VBAT
- net col1 renamed l_col1
- net col2 renamed l_col2
- net col3 renamed l_col3
- net col4 renamed l_col4
- net col5 renamed l_col5
- net row1 renamed l_row1
- net row2 renamed l_row2
- net row3 renamed l_row3
- net row4 renamed l_row4
Routing:
- net l_col1: track 155.9 -> 154.5 mm
- net l_row3: track 162.4 -> 163.4 mm
- net l_row2: track 159.9 -> 160.8 mm
- net l_BAT+: track 46.9 -> 47.7 mm
- net l_row1: track 164.4 -> 165.2 mm
- net l_RESET: track 24.6 -> 25.1 mm
Other:
- board size 114.3 x 93 mm -> 248.9 x 93.1 mm

Commit message: wip
Parts:
- BAT+2, BATGND2, r_D1, r_D10, r_D11, r_D12, r_D13, r_D14, r_D15, r_D16, r_D17, r_D2, r_D3, r_D4, r_D5, r_D6, r_D7, r_D8, r_D9: moved to B.Cu
- moved r_D5 114.2 mm to (197.2, 57.4)
- moved r_D4 104.5 mm to (215.4, 54.3)
- moved r_D10 103.9 mm to (196.8, 74.8)
- moved r_D17 101.9 mm to (180.8, 122.2)
- moved r_D3 99.9 mm to (234.1, 48.3)
- moved BAT+2 98.3 mm to (202.4, 82.6), turned to 180 degrees
- moved BATGND2 98.3 mm to (202.4, 86.1), turned to 180 degrees
- moved r_D15 96.6 mm to (197.2, 92.1)
- moved r_D9 91.2 mm to (215.4, 72.2)
- moved r_D2 86.8 mm to (252.4, 54.5)
- moved r_D16 84.9 mm to (201.6, 111.4)
- moved r_D8 84.2 mm to (234.1, 65.5)
- moved r_D14 81.7 mm to (215.3, 89.5)
- moved r_sw11 74.7 mm to (267.4, 100.5)
- moved r_sw10 74.7 mm to (193.3, 73.9)
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Routing:
- net r_col1: track 0.00 -> 138.6 mm, vias 0 -> 1
- net r_row1: track 0.00 -> 126.1 mm
- net r_col2: track 0.00 -> 123.9 mm, vias 0 -> 2
- net r_col3: track 0.00 -> 115.0 mm, vias 0 -> 3
- net r_row3: track 0.00 -> 95.5 mm
- net r_col4: track 0.00 -> 87.6 mm, vias 0 -> 3
- net r_row2: track 0.00 -> 85.7 mm
- net r_col5: track 0.00 -> 56.7 mm, vias 0 -> 1
- net r_GND: track 0.00 -> 56.2 mm, vias 0 -> 1
- net r_row4: track 0.00 -> 41.6 mm
- net r_BAT+: track 0.00 -> 39.6 mm
- net r_VBAT: track 0.00 -> 33.2 mm, vias 0 -> 2
- net r_RESET: track 0.00 -> 19.0 mm, vias 0 -> 1
- net Net-(r_D13-K): track 0.00 -> 16.1 mm, vias 0 -> 1
- net Net-(r_D17-K): track 0.00 -> 5.47 mm, vias 0 -> 1
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
Commit message: v1?
Parts:
- added ?: , , F.Cu at (193.8, 65.5)
- added ?: , , F.Cu at (267.2, 91.4)
- added ?: , , F.Cu at (238.8, 55.5)
- added ?: , , F.Cu at (181.0, 123.2)
- added REF**: PEM_SMTSO-M2-3ET, chocopi:PEM_SMTSO-M2-3ET, B.Cu at (110.3, 65.5)
- added REF**: PEM_SMTSO-M2-3ET, chocopi:PEM_SMTSO-M2-3ET, B.Cu at (36.9, 91.4)
- added REF**: PEM_SMTSO-M2-3ET, chocopi:PEM_SMTSO-M2-3ET, B.Cu at (123.1, 123.2)
- added REF**: PEM_SMTSO-M2-3ET, chocopi:PEM_SMTSO-M2-3ET, B.Cu at (65.3, 55.5)
- moved r_D17 11.0 mm to (174.7, 113.1)
Routing:
- net l_VBAT: track 28.7 -> 24.8 mm
- net l_col5: track 46.9 -> 50.0 mm
- net Net-(r_D17-K): track 5.47 -> 8.04 mm
- net l_row1: track 165.2 -> 162.7 mm
- net l_col1: track 154.5 -> 152.2 mm
- net r_col1: track 138.6 -> 140.9 mm
- net r_col5: track 56.7 -> 57.8 mm
- net r_row4: track 41.6 -> 42.2 mm

Commit message: mousebites!
Parts:
- added REF**: mousebites 2mm, chocopi:mousebites_2.5mm, F.Cu at (183.7, 76.7)
- added REF**: mousebites 2mm, chocopi:mousebites_2.5mm, F.Cu at (120.6, 60.7)
- added REF**: mousebites 2mm, chocopi:mousebites_2.5mm, F.Cu at (183.7, 60.7)
- added REF**: mousebites 2mm, chocopi:mousebites_2.5mm, F.Cu at (120.6, 76.7)
